File: I2C/16*Vibrationdriver.sch (EAGLE design)
At the start: 32 parts, among them IC1 LM317MDTRKG, U1 PCA9685, U2 ULN2803ADWR, U3 ULN2803ADWR

Commit message: Updates
Parts:
- removed C_V3: 100µ, thar:CAPACITOR1206
- removed JP10, JP9: (no value), pinhead:PINHD-1X9
- removed JP3, JP4: (no value), pinhead:PINHD-1X5
- removed RA0D, RA1D, RA2D, RA3D, RA4D, RA5D: 10k, thar:RESISTOR0603
- removed RA0U, RA1U, RA2U, RA3U, RA4U, RA5U, R_0: 0, thar:RESISTOR0603
- added A0, A1, A2, A3, A4, A5: (no value), SparkFun-Retired:SOLDERJUMPER_2WAYPASTE2&3
- added GND, SCL, SDA, TP1, TP10, TP11, TP12, TP13, TP14, TP15, TP16, TP17, TP18, TP19, TP2, TP20, TP21, TP22, TP23, TP24, TP25, TP26, TP27, TP28, TP29, TP3, TP30, TP31, TP32, TP4, TP5, TP6, TP7, TP8, TP9, VIN: TPTP16SQ, testpad:TPTP16SQ
- C_V2: value 100n -> 100µ; device thar:CAPACITOR -> thar:CAPACITOR1206
- R_VD: value 5k? -> 820
- R_VU: value 121? -> 470
Connections:
- removed net A0: RA0D.1, RA0U.2, U1.A0
- removed net A1: RA1D.1, RA1U.2, U1.A1
- removed net A2: RA2D.1, RA2U.2, U1.A2
- removed net A3: RA3D.1, RA3U.2, U1.A3
- removed net A4: RA4D.1, RA4U.2, U1.A4
- removed net A5: RA5D.1, RA5U.2, U1.A5
- new net N$3: A4.2, U1.A4
- new net N$4: A3.2, U1.A3
- new net N$5: A2.2, U1.A2
- new net N$6: A1.2, U1.A1
- new net N$7: A0.2, U1.A0
- net +3V3: now also A0.1, A1.1, A2.1, A3.1, A4.1, A5.1, LED1.A, TP17.TP, TP18.TP, TP19.TP, TP20.TP, TP21.TP, TP22.TP, TP23.TP, TP24.TP, TP25.TP, TP26.TP, TP27.TP, TP28.TP, TP29.TP, TP30.TP, TP31.TP, TP32.TP, U1.VDD; no longer C_V3.2, JP10.9, JP9.9, RA0U.1, RA1U.1, RA2U.1, RA3U.1, RA4U.1, RA5U.1, R_0.1
- net GND: now also A0.3, A1.3, A2.3, A3.3, A4.3, A5.3, GND.TP; no longer C_V3.1, JP3.5, JP4.5, RA0D.2, RA1D.2, RA2D.2, RA3D.2, RA4D.2, RA5D.2
- net N$14: now also TP1.TP; no longer JP10.1
- net N$19: now also TP2.TP; no longer JP10.2
- net N$2: now also A5.2, U1.A5; no longer R_0.2, U1.VDD
- net N$20: now also TP3.TP; no longer JP10.3
- net N$21: now also TP4.TP; no longer JP10.4
- net N$22: now also TP5.TP; no longer JP10.5
- net N$23: now also TP6.TP; no longer JP10.6
- net N$24: now also TP7.TP; no longer JP10.7
- net N$25: now also TP8.TP; no longer JP10.8
- net N$26: now also TP9.TP; no longer JP9.1
- net N$27: now also TP10.TP; no longer JP9.2
- net N$28: now also TP11.TP; no longer JP9.3
- net N$29: now also TP12.TP; no longer JP9.4
- net N$30: now also TP13.TP; no longer JP9.5
- net N$31: now also TP14.TP; no longer JP9.6
- net N$32: now also TP15.TP; no longer JP9.7
- net N$33: now also TP16.TP; no longer JP9.8
- net OE: no longer JP3.4, JP4.4
- net SCL: now also SCL.TP; no longer JP3.3, JP4.3
- net SDA: now also SDA.TP; no longer JP3.2, JP4.2
- net VCC: now also VIN.TP; no longer JP3.1, JP4.1, LED1.A
Other:
- moved on the sheet: C_MC, C_V2, R_RST
